File: PCB/pcb2molex8878_max.kicad_pcb (KiCad board)
At the start: 2 copper layers, 16.7 x 39.8 mm, 5 parts

Commit message: supply all files for all variants
Parts:
- removed REF** (x4): MountingHole_2.2mm_M2, Mounting_Holes:MountingHole_2.2mm_M2
- added J?: pcb2molex8878_max, 000_LOCAL:pcb2molex8878_max, F.Cu at (147.2, 99.2)
Changed lines of the file:
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@@
   (general
     (thickness 1.6)
-    (drawings 35)
+    (drawings 33)
     (tracks 0)
     (zones 0)
-    (modules 5)
+    (modules 2)
     (nets 1)
   )
@@
       (drillshape 0)
       (scaleselection 1)
-      (outputdirectory "gerber/"))
+      (outputdirectory "gerber_export/max/"))
   )
   (net 0 "")
@@
     (diff_pair_gap 0.254)
   )
-  (module 000_LOCAL:pcb2molex8878 (layer Top)
+  (module 000_LOCAL:pcb2molex8878_max (layer Top)
+    (at 147.2184 99.187)
+    (descr "Castellated edge contacts to fit Molex 8878 Socket")
+    (solder_mask_margin -0.28)
+    (fp_text reference J? (at -0.9906 -0.9906 -90) (layer Dwgs.User) hide
+      (effects (font (size 1.2065 1.2065) (thickness 0.127)) (justify left bottom))
+    )
+    (fp_text value pcb2molex8878_max (at 2.23 -9.45 -90) (layer F.Fab) hide
+      (effects (font (size 1.2065 1.2065) (thickness 0.1016)) (justify left bottom))
+    )
+    (fp_line (start -6.35 19.1) (end 6.35 19.1) (layer Eco2.User) (width 0.01))
+    (fp_line (start -8.35 19.9) (end -6.35 19.9) (layer Eco2.User) (width 0.01))
+    (fp_line (start 8.35 19.9) (end 6.35 19.9) (layer Eco2.User) (width 0.01))
+    (fp_line (start -4.35 -19.1) (end 6.35 -19.1) (layer Eco2.User) (width 0.01))
+    (fp_line (start 8.35 -19.9) (end 6.35 -19.9) (layer Eco2.User) (width 0.01))
+    (fp_line (start -8.35 -19.9) (end -4.35 -19.9) (layer Eco2.User) (width 0.01))
+    (fp_line (start -8.35 -19.1) (end 8.35 19.1) (layer Dwgs.User) (width 0.01))
+    (fp_line (start -8.35 19.1) (end 8.35 -19.1) (layer Dwgs.User) (width 0.01))
+    (fp_text user "Eco2.User is Edge.Cuts for use with \"pcb2molex8878_max\" carrier." (at -0.18 13.04) (layer Eco2.User)
+      (effects (font (size 0.2 0.2) (thickness 0.01)))
+    )
+    (fp_line (start -8.35 -19.9) (end -8.35 19.9) (layer Eco2.User) (width 0.01))
+    (fp_line (start 8.35 19.9) (end 8.35 -19.9) (layer Eco2.User) (width 0.01))
+    (fp_line (start -6.35 19.1) (end -6.35 19.9) (layer Eco2.User) (width 0.01))
+    (fp_line (start 6.35 19.9) (end 6.35 19.1) (layer Eco2.User) (width 0.01))
+    (fp_line (start 6.35 -19.1) (end 6.35 -19.9) (layer Eco2.User) (width 0.01))
+    (fp_line (start -4.35 -19.9) (end -4.35 -19.1) (layer Eco2.User) (width 0.01))
+    (pad "" np_thru_hole circle (at 6.35 19.45) (size 0.7 0.7) (drill 0.7) (layers *.Cu))
+    (pad "" np_thru_hole circle (at -6.35 19.45) (size 0.7 0.7) (drill 0.7) (layers *.Cu))
+    (pad "" np_thru_hole circle (at 6.35 -19.45) (size 0.7 0.7) (drill 0.7) (layers *.Cu))
+    (pad "" np_thru_hole circle (at -4.35 -19.45) (size 0.7 0.7) (drill 0.7) (layers *.Cu))
+    (model ${KIPRJMOD}/000_LOCAL.pretty/3d/pcb2molex8878_max.step
+      (offset (xyz 0 0 -0.4))
+      (scale (xyz 1 1 1))
+      (rotate (xyz 0 0 90))
+    )
+  )
+  (module 000_LOCAL:pcb2molex8878 locked (layer Top)
     (at 147.2184 99.187)
     (descr "Castellated edge contacts to fit Molex 8878 Socket")
@@
     (pad 1 thru_hole roundrect (at -8.6 -16.51) (size 1.8 1.6) (drill 1.6 (offset 0.1 0)) (layers *.Cu *.Mask) (roundrect_rratio 0.1)
       (solder_mask_margin -0.19))
-    (model ${KIPRJMOD}/000_LOCAL.pretty/3d/pcb2molex8878.step
-      (offset (xyz 0 0 -0.4))
-      (scale (xyz 1 1 1))
-      (rotate (xyz 0 0 90))
-    )
-  )
-  (module Mounting_Holes:MountingHole_2.2mm_M2 (layer Top)
-    (at 140.8684 118.637)
-    (descr "Mounting Hole 2.2mm, no annular, M2")
-    (tags "mounting hole 2.2mm no annular m2")
-    (attr virtual)
-    (fp_text reference REF** (at 0 -3.2) (layer F.SilkS) hide
-      (effects (font (size 1 1) (thickness 0.15)))
-    )
-    (fp_text value MountingHole_2.2mm_M2 (at 0 3.2) (layer F.Fab)
-      (effects (font (size 1 1) (thickness 0.15)))
-    )
-    (fp_text user %R (at 0.3 0) (layer F.Fab)
-      (effects (font (size 1 1) (thickness 0.15)))
-    )
-    (fp_circle (center 0 0) (end 2.2 0) (layer Cmts.User) (width 0.15))
-    (fp_circle (center 0 0) (end 2.45 0) (layer F.CrtYd) (width 0.05))
-    (pad "" np_thru_hole circle (at 0 0) (size 0.7 0.7) (drill 0.7) (layers *.Cu *.Mask))
-  )
-  (module Mounting_Holes:MountingHole_2.2mm_M2 (layer Top)
-    (at 153.5684 118.637)
-    (descr "Mounting Hole 2.2mm, no annular, M2")
-    (tags "mounting hole 2.2mm no annular m2")
-    (attr virtual)
-    (fp_text reference REF** (at 0 -3.2) (layer F.SilkS) hide
-      (effects (font (size 1 1) (thickness 0.15)))
-    )
-    (fp_text value MountingHole_2.2mm_M2 (at 0 3.2) (layer F.Fab)
-      (effects (font (size 1 1) (thickness 0.15)))
-    )
-    (fp_circle (center 0 0) (end 2.45 0) (layer F.CrtYd) (width 0.05))
-    (fp_circle (center 0 0) (end 2.2 0) (layer Cmts.User) (width 0.15))
-    (fp_text user %R (at 0.3 0) (layer F.Fab)
-      (effects (font (size 1 1) (thickness 0.15)))
-    )
-    (pad "" np_thru_hole circle (at 0 0) (size 0.7 0.7) (drill 0.7) (layers *.Cu *.Mask))
-  )
-  (module Mounting_Holes:MountingHole_2.2mm_M2 (layer Top)
-    (at 153.5684 79.737)
-    (descr "Mounting Hole 2.2mm, no annular, M2")
-    (tags "mounting hole 2.2mm no annular m2")
-    (attr virtual)
-    (fp_text reference REF** (at 0 -3.2) (layer F.SilkS) hide
-      (effects (font (size 1 1) (thickness 0.15)))
-    )
-    (fp_text value MountingHole_2.2mm_M2 (at 0 3.2) (layer F.Fab)
-      (effects (font (size 1 1) (thickness 0.15)))
-    )
-    (fp_text user %R (at 0.3 0) (layer F.Fab)
-      (effects (font (size 1 1) (thickness 0.15)))
-    )
-    (fp_circle (center 0 0) (end 2.2 0) (layer Cmts.User) (width 0.15))
-    (fp_circle (center 0 0) (end 2.45 0) (layer F.CrtYd) (width 0.05))
-    (pad "" np_thru_hole circle (at 0 0) (size 0.7 0.7) (drill 0.7) (layers *.Cu *.Mask))
-  )
-  (module Mounting_Holes:MountingHole_2.2mm_M2 (layer Top)
-    (at 142.8684 79.737)
-    (descr "Mounting Hole 2.2mm, no annular, M2")
-    (tags "mounting hole 2.2mm no annular m2")
-    (attr virtual)
-    (fp_text reference REF** (at 0 -3.2) (layer F.SilkS) hide
-      (effects (font (size 1 1) (thickness 0.15)))
-    )
-    (fp_text value MountingHole_2.2mm_M2 (at 0 3.2) (layer F.Fab)
-      (effects (font (size 1 1) (thickness 0.15)))
-    )
-    (fp_circle (center 0 0) (end 2.45 0) (layer F.CrtYd) (width 0.05))
-    (fp_circle (center 0 0) (end 2.2 0) (layer Cmts.User) (width 0.15))
-    (fp_text user %R (at 0.3 0) (layer F.Fab)
-      (effects (font (size 1 1) (thickness 0.15)))
-    )
-    (pad "" np_thru_hole circle (at 0 0) (size 0.7 0.7) (drill 0.7) (layers *.Cu *.Mask))
-  )
+  )
+  (dimension 4.000001 (width 0.0127) (layer Dwgs.User)
+    (gr_text "       4.00" (at 140.868399 76.4544) (layer Dwgs.User)
+      (effects (font (size 0.4572 0.4572) (thickness 0.0127)) (justify left))
+    )
+    (feature1 (pts (xy 142.868401 79.286999) (xy 142.8684 76.350579)))
+    (feature2 (pts (xy 138.8684 79.287) (xy 138.868399 76.35058)))
+    (crossbar (pts (xy 138.868399 76.937001) (xy 142.8684 76.937)))
+    (arrow1a (pts (xy 142.8684 76.937) (xy 141.741896 77.523421)))
+    (arrow1b (pts (xy 142.8684 76.937) (xy 141.741896 76.35058)))
+    (arrow2a (pts (xy 138.868399 76.937001) (xy 139.994903 77.523421)))
+    (arrow2b (pts (xy 138.868399 76.937001) (xy 139.994903 76.35058)))
+  )
+  (gr_line (start 138.8684 119.087) (end 138.8684 79.287) (layer Edge.Cuts) (width 0.0254))
+  (gr_line (start 138.8684 119.087) (end 140.8684 119.087) (layer Edge.Cuts) (width 0.0254))
+  (gr_line (start 140.8684 119.087) (end 140.8684 118.287) (layer Edge.Cuts) (width 0.0254))
   (gr_line (start 141.2184 118.237) (end 141.4184 118.037) (layer Dwgs.User) (width 0.0127))
   (gr_line (start 141.2184 118.237) (end 141.0184 118.037) (layer Dwgs.User) (width 0.0127))
@@
   )
   (dimension 0.7 (width 0.0127) (layer Dwgs.User)
-    (gr_text "   0.70 diameter" (at 142.8684 81.9696) (layer Dwgs.User)
+    (gr_text "   0.70" (at 142.8684 81.9696) (layer Dwgs.User)
       (effects (font (size 0.4572 0.4572) (thickness 0.0127)) (justify left))
     )
@@
     (arrow2b (pts (xy 153.5684 76.937) (xy 154.694904 76.350579)))
   )
-  (dimension 4.000001 (width 0.0127) (layer Dwgs.User)
-    (gr_text "       4.00" (at 140.868399 76.4544) (layer Dwgs.User)
-      (effects (font (size 0.4572 0.4572) (thickness 0.0127)) (justify left))
-    )
-    (feature1 (pts (xy 142.868401 79.286999) (xy 142.8684 76.350579)))
-    (feature2 (pts (xy 138.8684 79.287) (xy 138.868399 76.35058)))
-    (crossbar (pts (xy 138.868399 76.937001) (xy 142.8684 76.937)))
-    (arrow1a (pts (xy 142.8684 76.937) (xy 141.741896 77.523421)))
-    (arrow1b (pts (xy 142.8684 76.937) (xy 141.741896 76.35058)))
-    (arrow2a (pts (xy 138.868399 76.937001) (xy 139.994903 77.523421)))
-    (arrow2b (pts (xy 138.868399 76.937001) (xy 139.994903 76.35058)))
-  )
-  (gr_line (start 138.8684 119.087) (end 155.5684 79.287) (layer Dwgs.User) (width 0.0127))
-  (gr_line (start 138.8684 79.287) (end 155.5684 119.087) (layer Dwgs.User) (width 0.0127))
   (gr_arc (start 152.7084 79.227) (end 152.7084 80.087) (angle -86.0090869) (layer Dwgs.User) (width 0.0127))
   (gr_arc (start 143.728401 79.224911) (end 142.868402 79.28491) (angle -86.0090869) (layer Dwgs.User) (width 0.0127))
@@
   (gr_line (start 138.8684 79.287) (end 142.8684 79.287) (layer Edge.Cuts) (width 0.0254))
   (gr_line (start 153.5684 79.287) (end 155.5684 79.287) (layer Edge.Cuts) (width 0.0254))
-  (gr_line (start 138.8684 119.087) (end 138.8684 79.287) (layer Edge.Cuts) (width 0.0254))
   (gr_line (start 155.5684 119.087) (end 155.5684 79.287) (layer Edge.Cuts) (width 0.0254))
   (gr_line (start 140.8684 118.287) (end 153.5684 118.287) (layer Edge.Cuts) (width 0.0254))
   (gr_line (start 153.5684 119.087) (end 155.5684 119.087) (layer Edge.Cuts) (width 0.0254))
   (gr_line (start 153.5684 118.287) (end 153.5684 119.087) (layer Edge.Cuts) (width 0.0254))
-  (gr_line (start 140.8684 119.087) (end 140.8684 118.287) (layer Edge.Cuts) (width 0.0254))
-  (gr_line (start 138.8684 119.087) (end 140.8684 119.087) (layer Edge.Cuts) (width 0.0254))
 )
