File: PCB/Molex78802_PCB_28.kicad_pcb (KiCad board)
At the start: 2 copper layers, 16.5 x 38 mm, 1 part

Commit message: Rename to Molex78802. Add DIP variant. Add 24 and 32 pin versions.
Parts:
- J?: value Molex78805_PCB -> Molex78802_PCB_28; footprint 000_LOCAL:Molex78805_PCB -> 000_LOCAL:Molex78802_PCB_28
Changed lines of the file:
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@@
-(kicad_pcb (version 20171130) (host pcbnew 5.1.9-73d0e3b20d~88~ubuntu20.10.1)
+(kicad_pcb (version 20171130) (host pcbnew 5.1.10-88a1d61d58~88~ubuntu20.10.1)
   (general
     (thickness 1.6)
@@
   (page A4)
   (title_block
-    (title "PCB to Fit Inside Molex 15-29-9282 Socket")
-    (date 2021-03-16)
-    (rev 002)
+    (title "Molex78802 PCB 28")
+    (date 2021-05-20)
+    (rev 003)
     (company b.kenyon.w@gmail.com)
   )
@@
     (diff_pair_gap 0.254)
   )
-  (module 000_LOCAL:Molex78805_PCB (layer Top)
+  (module 000_LOCAL:Molex78802_PCB_28 (layer Top)
     (at 147.2184 99.187)
     (descr "Castellated edge contacts to fit Molex 78805 Socket")
@@
       (effects (font (size 1.2065 1.2065) (thickness 0.127)) (justify bottom))
     )
-    (fp_text value Molex78805_PCB (at 1.27 0 -90) (layer F.Fab) hide
+    (fp_text value Molex78802_PCB_28 (at 1.27 0 -90) (layer F.Fab) hide
       (effects (font (size 1.2065 1.2065) (thickness 0.1016)) (justify bottom))
     )
@@
       (zone_connect 0))
     (pad 15 thru_hole circle (at 8.5552 16.51 180) (size 1.6002 1.6002) (drill 1.59766) (layers *.Cu *.Mask))
-    (model ${KIPRJMOD}/000_LOCAL.pretty/3d/Molex78805_PCB_Carrier_chamfer.step
-      (offset (xyz 0 0 -0.25))
+    (model ${KIPRJMOD}/000_LOCAL.pretty/3d/Molex78802_PCB_28.step
+      (offset (xyz 0 0 -0.18))
       (scale (xyz 1 1 1))
       (rotate (xyz 0 0 90))
